File: Wago 859-SSD.kicad_pcb (KiCad board)
At the start: 2 copper layers, 74.3 x 51.3 mm, 17 parts, among them J1 IN+, J2 IN-, J3 OUT VB, J5 OUT+, J8 OUT1-, Q2 BSS138, Q3 BSS84, U1 PC817

Commit message: Bugfix Version: V3
Parts:
- removed JP2: SolderJumper_3_Open, Jumper:SolderJumper-3_P1.3mm_Open_Pad1.0x1.5mm
- removed Q2: BSS138, Package_TO_SOT_SMD:SOT-23_Handsoldering
- removed the R4 at (36.8, 29.1)
- renumbered Q3 to Q1, R6 to R1, R3 to R2, R2 to R3, R5 to R4
Connections:
- Q1 pad 1: Net-(Q2-D) -> Net-(Q1-G)
- R1 pad 1: Net-(Q2-D) -> Net-(Q1-G)
- R2 pad 1: GND -> Net-(R2-Pad1)
- R2 pad 2: Net-(Q2-S) -> Net-(Q1-G)
- R4 pad 1: Net-(JP2-B) -> Net-(D1-A)
- U1 pad 3: Net-(Q2-S) -> GND
- U1 pad 4: Net-(Q2-D) -> Net-(R2-Pad1)
Routing:
- net Net-(Q2-D): track 23.6 -> 0.00 mm
- net Net-(Q2-S): track 19.6 -> 0.00 mm, vias 2 -> 0
- net Net-(JP2-A): track 18.5 -> 0.00 mm
- net Net-(R2-Pad1): track 0.00 -> 10.7 mm
- net Net-(Q1-G): track 0.00 -> 8.65 mm
- net Net-(JP2-B): track 3.91 -> 0.00 mm
- net Net-(D1-A): track 35.2 -> 37.3 mm
Other:
- board text added: "Wago 859-SSD V3"
